File: zuul.kicad_pcb (KiCad board)
At the start: 2 copper layers, 17.8 x 55.9 mm, 8 parts, among them IC1 DRV8251DDAR, J1 Raspberry_Pi_2_3, J2 MOTOR_OUTPUT, J5 Conn_01x06_Male

Commit message: ummm
Routing:
- net /LED_GPIO: track 8.47 -> 12.6 mm
