File: zuul.kicad_sch (KiCad schematic)
At the start: 6 parts, among them IC1 DRV8251DDAR, J1 Raspberry_Pi_2_3, J2 MOTOR_OUTPUT

Commit message: compuger
Parts:
- added C3: 47μF, Capacitor_SMD:C_0805_2012Metric, symbol Device:C
- added J5: Conn_01x06_Male, Connector_JST:JST_XH_S6B-XH-A_1x06_P2.50mm_Horizontal, symbol TalDoor-rescue:Conn_01x06_Male
- C1: value 0.1uF -> 0.1μF; footprint (none) -> Capacitor_SMD:C_0402_1005Metric
- C2: value C_BULK -> 47μF; footprint (none) -> Capacitor_SMD:C_0805_2012Metric
- J1: footprint (none) -> Connector_PinSocket_2.54mm:PinSocket_2x20_P2.54mm_Vertical
- J2: footprint (none) -> Library:CUSTOM_PIN_HEADER_01x02_J2
- R1: value R_SENSE -> 6.5Ω; footprint (none) -> Resistor_SMD:R_1206_3216Metric
Connections:
- net GND: now also C3.2, J5.2 (Pin_2)
- net MOTOR_BACKWARD: now also J1.13 (GPIO27); no longer J1.19 (MOSI0/GPIO10)
- net MOTOR_FORWARD: now also J1.15 (GPIO22); no longer J1.21 (MISO0/GPIO9)
- net VCC: now also C3.1, J5.1 (Pin_1); no longer IC1.4 (VREF)
- net +3V3: now reaches J1.1 (3V3)
- net +3V3: now also IC1.4 (VREF), J1.17 (3V3)
- net RXD: now reaches J1.10 (GPIO15/RXD)
- net RXD: now also J5.5 (Pin_5)
- net BEEPER: now reaches J1.12 (GPIO18/PWM0)
- net BEEPER: now also J5.4 (Pin_4)
- net LED_GPIO: now reaches J1.31 (GCLK2/GPIO6)
- net LED_GPIO: now also J5.3 (Pin_3)
- net TXD: now reaches J1.8 (GPIO14/TXD)
- net TXD: now also J5.6 (Pin_6)
Other:
- moved on the sheet: J2
